File: USAR_Drone_Feature.kicad_pcb (KiCad board)
At the start: 2 copper layers, 50 x 50 mm, 0 parts

Commit message: pcb desing done, add productions files
Parts:
- added C1: 10uF/10V, PCM_Capacitor_SMD_AKL:C_0805_2012Metric, F.Cu at (216.3, 89.8)
- added C10: 100nF 25V, PCM_Capacitor_SMD_AKL:C_0603_1608Metric, F.Cu at (182.3, 90.6)
- added C11: 3.3nF 25V, PCM_Capacitor_SMD_AKL:C_0603_1608Metric, F.Cu at (185.8, 90.1)
- added C12: 22uF 25V, PCM_Capacitor_SMD_AKL:C_0805_2012Metric, F.Cu at (183.1, 102.1)
- added C13: 22uF 25V, PCM_Capacitor_SMD_AKL:C_0805_2012Metric, F.Cu at (185.8, 98.6)
- added C2: 100nF 25V, PCM_Capacitor_SMD_AKL:C_0603_1608Metric, F.Cu at (199.3, 92.1)
- added C3: 1uF 25V, PCM_Capacitor_SMD_AKL:C_0805_2012Metric, F.Cu at (201.6, 92.1)
- added C4: 1uF 25V, PCM_Capacitor_SMD_AKL:C_0805_2012Metric, F.Cu at (224.3, 118.3)
- added C5: 100nF 25V, PCM_Capacitor_SMD_AKL:C_0603_1608Metric, F.Cu at (219.6, 126.3)
- added C6: 100nF 25V, PCM_Capacitor_SMD_AKL:C_0603_1608Metric, F.Cu at (197.6, 109.6)
- added C7: 100nF 25V, PCM_Capacitor_SMD_AKL:C_0603_1608Metric, F.Cu at (219.8, 119.6)
- added C8: 10uF 25V, PCM_Capacitor_SMD_AKL:C_1210_3225Metric, F.Cu at (178.8, 99.1)
- added C9: 10uF 25V, PCM_Capacitor_SMD_AKL:C_1210_3225Metric, F.Cu at (178.8, 105.6)
- added D1: B0540W, EasyEDA:SOD-123_L2.7-W1.6-LS3.7-FD, F.Cu at (214.8, 86.3)
- added D2: ESD5B5.0S, PCM_Diode_SMD_AKL:D_SOD-523, F.Cu at (224.1, 106.6)
- added D3: ESD5B5.0S, PCM_Diode_SMD_AKL:D_SOD-523, F.Cu at (217.3, 106.8)
- added D4: ESD5Z3.3T, PCM_Diode_SMD_AKL:D_SOD-523, F.Cu at (221.6, 116.6)
- added D5: ESD5Z3.3T, PCM_Diode_SMD_AKL:D_SOD-523, F.Cu at (216.6, 101.8)
- added D6: SS24-SMB, EasyEDA:SMB_L4.3-W3.6-LS5.3-RD, F.Cu at (179.0, 92.2)
- added H1: MountingHole, MountingHole:MountingHole_2.2mm_M2_DIN965, F.Cu at (201.1, 87.8)
- added H2: MountingHole, MountingHole:MountingHole_2.2mm_M2_DIN965, F.Cu at (179.6, 126.8)
- added H3: MountingHole, MountingHole:MountingHole_2.2mm_M2_DIN965, F.Cu at (223.3, 126.8)
- added H4: MountingHole, MountingHole:MountingHole_2.2mm_M2_DIN965, F.Cu at (223.1, 83.3)
- added J1: DB128L-5.08-2P-BK-S, EasyEDA:CONN-TH_2P-P5.08_DB128L-5.08-2P-BK-S, F.Cu at (181.8, 83.1)
- added J2: DB128L-5.08-2P-BK-S, EasyEDA:CONN-TH_2P-P5.08_DB128L-5.08-2P-BK-S, F.Cu at (193.3, 83.1)
- added J3: Conn_02x04_Odd_Even, Connector_PinHeader_2.54mm:PinHeader_2x04_P2.54mm_Vertical, F.Cu at (179.1, 113.3)
- added J4: Conn_01x04_Socket, EasyEDA:CONN-TH_B4B-PH-K-S, F.Cu at (204.0, 82.9)
- added J5: Conn_01x04_Socket, EasyEDA:CONN-TH_B4B-PH-K-S, F.Cu at (215.0, 82.9)
- added J6: Conn_01x04_Socket, EasyEDA:CONN-TH_B4B-PH-K-S, F.Cu at (190.8, 127.2)
- added JP1: SolderJumper_2_Open, PCM_SparkFun-Jumper:Jumper_2_NO, F.Cu at (206.3, 86.3)
- added JP2: SolderJumper_2_Open, PCM_SparkFun-Jumper:Jumper_2_NO, F.Cu at (208.6, 86.3)
- added JP3: SolderJumper_2_Open, PCM_SparkFun-Jumper:Jumper_2_NO, F.Cu at (188.8, 102.8)
- added JP4: SolderJumper_2_Open, PCM_SparkFun-Jumper:Jumper_2_NO, F.Cu at (194.6, 99.6)
- added L1: MDMK2020T2R2MM, Snapeda:IND_MDMK2020T1R0MM_TAY, F.Cu at (187.1, 105.8)
- added L2: SRP4020TA-2R2M, Snapeda:IND_SRP4020TA_BRN-L, F.Cu at (190.6, 96.3)
- added LED1: XL-1608SURC-06, EasyEDA:LED0603-RD_RED, F.Cu at (210.6, 101.1)
- added LED2: XL-1608SURC-06, EasyEDA:LED0603-RD_RED, F.Cu at (212.8, 101.1)
- added R1: 5.1K, PCM_Resistor_SMD_AKL:R_0603_1608Metric, F.Cu at (221.8, 98.3)
- added R10: 10K, PCM_Resistor_SMD_AKL:R_0603_1608Metric, F.Cu at (185.1, 114.3)
- added R11: 10K, PCM_Resistor_SMD_AKL:R_0603_1608Metric, F.Cu at (187.8, 114.3)
- added R13: 2.2K, PCM_Resistor_SMD_AKL:R_0603_1608Metric, F.Cu at (193.3, 121.3)
- added R14: 2.2K, PCM_Resistor_SMD_AKL:R_0603_1608Metric, F.Cu at (196.1, 121.3)
- added R15: 2.2K, PCM_Resistor_SMD_AKL:R_0603_1608Metric, F.Cu at (208.8, 105.6)
- added R16: 2.2K, PCM_Resistor_SMD_AKL:R_0603_1608Metric, F.Cu at (205.8, 105.6)
- added R17: 10K, PCM_Resistor_SMD_AKL:R_0603_1608Metric, F.Cu at (194.8, 109.5)
- added R18: 10K, PCM_Resistor_SMD_AKL:R_0603_1608Metric, F.Cu at (222.5, 122.1)
- added R19: 10K, PCM_Resistor_SMD_AKL:R_0603_1608Metric, F.Cu at (184.5, 126.5)
- added R2: 5.1K, PCM_Resistor_SMD_AKL:R_0603_1608Metric, F.Cu at (213.3, 89.6)
- added R20: 100k, PCM_Resistor_SMD_AKL:R_0603_1608Metric, F.Cu at (186.1, 108.8)
- added R21: 100k, PCM_Resistor_SMD_AKL:R_0603_1608Metric, F.Cu at (194.6, 95.1)
- added R3: 33R, PCM_Resistor_SMD_AKL:R_0603_1608Metric, F.Cu at (221.8, 107.8)
- added R4: 33R, PCM_Resistor_SMD_AKL:R_0603_1608Metric, F.Cu at (219.8, 107.8)
- added R5: 10K, PCM_Resistor_SMD_AKL:R_0603_1608Metric, F.Cu at (197.3, 92.0)
- added R6: 10K, PCM_Resistor_SMD_AKL:R_0603_1608Metric, F.Cu at (197.3, 95.6)
- added R7: 10K, PCM_Resistor_SMD_AKL:R_0603_1608Metric, F.Cu at (209.8, 98.3)
- added R8: 10K, PCM_Resistor_SMD_AKL:R_0603_1608Metric, F.Cu at (211.1, 95.3)
- added R9: 10K, PCM_Resistor_SMD_AKL:R_0603_1608Metric, F.Cu at (185.1, 121.6)
- added SW1: TS-1088-AR02016, EasyEDA:SW-SMD_L3.9-W3.0-P4.45, F.Cu at (222.6, 113.3)
- added SW2: TS-1088-AR02016, EasyEDA:SW-SMD_L3.9-W3.0-P4.45, F.Cu at (221.6, 102.6)
- added U1: ESP32-S3-WROOM-1(N16R8), EasyEDA:WIRELM-SMD_ESP32-S3-WROOM-1, F.Cu at (208.6, 118.1)
- added U2: TPS62172DSG, Package_SON:WSON-8-1EP_2x2mm_P0.5mm_EP0.9x1.6mm_ThermalVias, F.Cu at (183.1, 106.6)
- added U3: TPS62133, Package_DFN_QFN:VQFN-16-1EP_3x3mm_P0.5mm_EP1.68x1.68mm_ThermalVias, F.Cu at (185.3, 94.1)
- added USB1: TYPE-C 16PIN 2MD, EasyEDA:USB-C-SMD_TYPE-C-6PIN-2MD-073, F.Cu at (221.5, 91.6)
Routing:
- net +5V: track 0.00 -> 76.6 mm, vias 0 -> 5
- net /UART_P: track 0.00 -> 51.6 mm, vias 0 -> 2
- net /BATTERY2_LEVEL: track 0.00 -> 49.8 mm, vias 0 -> 2
- net /UART_N: track 0.00 -> 46.7 mm, vias 0 -> 2
- net /SERVO_PWM: track 0.00 -> 42.9 mm, vias 0 -> 1
- net /RST: track 0.00 -> 40.2 mm, vias 0 -> 2
- net GND: track 0.00 -> 39.0 mm, vias 0 -> 75
- net /IRQ: track 0.00 -> 39.0 mm, vias 0 -> 2
- net /I2C_P: track 0.00 -> 35.7 mm
- net /BOOT: track 0.00 -> 34.6 mm, vias 0 -> 2
- net /I2C_N: track 0.00 -> 34.4 mm
- net /DP: track 0.00 -> 22.4 mm
- net /CE: track 0.00 -> 21.7 mm
- net /MISO: track 0.00 -> 21.7 mm
- net /SCK: track 0.00 -> 21.5 mm
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- added copper zone on F.Cu, net +3V3
- added copper zone on In1.Cu, net +3V3
- added copper zone on F.Cu, net +5V
- added copper zone on F.Cu, net +7.5V
- added copper zone on F.Cu, net /PowerRails/L1
- added copper zone on F.Cu, net /PowerRails/L1_3V3
- added copper zone on F.Cu, net /PowerRails/Reg3v3_out
- added copper zone on F.Cu, net /PowerRails/Reg5v_out
- added copper zone on B.Cu, net GND
- added copper zone on F.Cu, net GND
- added copper zone on F.Cu, net Net-(J1-Pad2)
- added copper zone on F.Cu, net VCC
Other:
- copper layers 2 -> 4
- board text added: "BRECHA VIEJA V0.1"

Commit message: ajuste de agujeros
Parts:
- moved H3 0.50 mm to (222.8, 126.8)
Changed lines of the file:
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@@
 		(locked yes)
 		(layer "F.Cu")
-		(at 223.3 126.85)
+		(at 222.8 126.85)
 		(descr "Mounting Hole 2.2mm, M2, no annular, generated by kicad-footprint-generator mountinghole.py")
 		(tags "mountinghole M2 DIN965")
@@
 			(keep_text_aligned yes)
 		)
-		(gr_text "1968.5039"
+		(gr_text "50"
 			(at 244.15 105.1 90)
 			(layer "User.2")
@@
 			(keep_text_aligned yes)
 		)
-		(gr_text "1968.5039"
+		(gr_text "50"
 			(at 201.3 145.45 0)
 			(layer "User.2")

Commit message: ajuste de footprints, reposicionamiento de agujeros
Parts:
- removed J1, J2: DB128L-5.08-2P-BK-S, EasyEDA:CONN-TH_2P-P5.08_DB128L-5.08-2P-BK-S
- added CN1: B2B-XH-A, EasyEDA:CONN-TH_B2B-XH-A-LF-SN, F.Cu at (186.1, 83.1)
- added CN2: B2B-XH-A, EasyEDA:CONN-TH_B2B-XH-A-LF-SN, F.Cu at (194.3, 83.1)
- moved H1 22.0 mm to (179.6, 83.3)
- moved JP1 0.50 mm to (205.8, 86.3)
- moved H3 0.25 mm to (223.1, 126.8)
Routing:
- net +7.5V: track 19.3 -> 17.5 mm
- net VCC: track 7.36 -> 8.05 mm
- net Net-(J4-Pin_1): track 6.98 -> 7.48 mm
- added copper zone on F.Cu, net Net-(CN1-Pad2)
- removed copper zone on F.Cu, net Net-(J1-Pad2)
