File: USAR_Drone_Feature.kicad_sch (KiCad schematic)
At the start: 48 parts, among them CN1 B2B-XH-A, CN2 B2B-XH-A, J3 Conn_02x04_Odd_Even, J4 Conn_01x04_Socket, J5 Conn_01x04_Socket, J6 Conn_01x04_Socket, SW1 TS-1088-AR02016, SW2 TS-1088-AR02016, U1 ESP32-S3-WROOM-1(N16R8)

Commit message: cambio agujeros 2.2mm a 2.5mm
Parts:
- H1, H2, H3, H4: footprint MountingHole:MountingHole_2.2mm_M2_DIN965 -> MountingHole:MountingHole_2.5mm
Changed lines of the file:
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@@
 			)
 		)
-		(property "Footprint" "MountingHole:MountingHole_2.2mm_M2_DIN965"
+		(property "Footprint" "MountingHole:MountingHole_2.5mm"
 			(at 403.86 58.42 0)
 			(hide yes)
@@
 			)
 		)
-		(property "Footprint" "MountingHole:MountingHole_2.2mm_M2_DIN965"
+		(property "Footprint" "MountingHole:MountingHole_2.5mm"
 			(at 403.86 43.18 0)
 			(hide yes)
@@
 			)
 		)
-		(property "Footprint" "MountingHole:MountingHole_2.2mm_M2_DIN965"
+		(property "Footprint" "MountingHole:MountingHole_2.5mm"
 			(at 403.86 35.56 0)
 			(hide yes)
@@
 			)
 		)
-		(property "Footprint" "MountingHole:MountingHole_2.2mm_M2_DIN965"
+		(property "Footprint" "MountingHole:MountingHole_2.5mm"
 			(at 403.86 50.8 0)
 			(hide yes)

Commit message: cambiar bobina de power suppy
Other:
- title: (none) -> USARQ
Changed lines of the file:
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@@
 	(generator_version "10.0")
 	(paper "USLedger")
+	(title_block
+		(title "USARQ")
+		(rev "V0.1")
+	)
 	(text "MICRO"
 		(exclude_from_sim no)

Commit message: stable
Other:
- note added: "I2C"
- moved on the sheet: J3, J4, J5, J6, JP1, JP2, R10, R11, R19, R9
